File: yoring.kicad_pcb (KiCad board)
At the start: 4 copper layers, 31.1 x 50 mm, 65 parts, among them J1 USB-C_USB4105-GF-A, J3 Conn_01x05, SW1 SW_MEC_5E, SW2 SW_MEC_5E, U1 ESP32C3, U2 IS25LP016D-JLLE, U3 USBLC6-2SC6, U4 ICM-20602, U5 ICM-20602, U6 ICM-20602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

Commit message: Added a few things to layout
Parts:
- added kibuzzard-64F24942: G***, kibuzzard-64F24942, F.Cu at (115.5, 59.8)
- added kibuzzard-64F24971: G***, kibuzzard-64F24971, F.Cu at (94.9, 63.7)
- added kibuzzard-64F24993: G***, kibuzzard-64F24993, F.Cu at (94.9, 66.3)
- added kibuzzard-64F249A3: G***, kibuzzard-64F249A3, F.Cu at (94.9, 68.8)
- added kibuzzard-64F249B1: G***, kibuzzard-64F249B1, F.Cu at (94.9, 71.3)
- added kibuzzard-64F249BD: G***, kibuzzard-64F249BD, F.Cu at (94.9, 73.9)
Other:
- board text added: "YŌRING"
